Commit message: Record video 0725

File: oil_description/urdf/oil_description.urdf (robot description, URDF)
Before this commit: robot oil_description, 10 links, 9 joints
Joints:
- joint joint1: limit lower=-0.4 upper=0.4 effort=0 velocity=0 -> lower=-0.34 upper=0.34 effort=0 velocity=0
- joint joint2: limit lower=-1.500 upper=1.500 effort=0 velocity=0 -> lower=-0.000 upper=0.000 effort=0 velocity=0
- joint joint4: limit lower=-1.500 upper=1.500 effort=0 velocity=0 -> lower=-1.000 upper=1.000 effort=0 velocity=0
- joint joint6: limit lower=-1.500 upper=1.500 effort=0 velocity=0 -> lower=-1.000 upper=1.000 effort=0 velocity=0

Commit message: prepare for handeye calibration

File: oil_description/urdf/oil_description.urdf (robot description, URDF)
Before this commit: robot oil_description, 10 links, 9 joints
Joints:
- joint joint2: limit lower=-0.000 upper=0.000 effort=0 velocity=0 -> lower=-1.000 upper=1.000 effort=0 velocity=0

Commit message: add function of hmi: moveL reference to base_link or ee_link

File: oil_description/urdf/oil_description.urdf (robot description, URDF)
Before this commit: robot oil_description, 10 links, 9 joints
Joints:
- joint joint3: limit lower=-3.0 upper=3.0 effort=0 velocity=0 -> lower=-0.34 upper=0.34 effort=0 velocity=0

Commit message: add obstacles to urdf

File: oil_description/urdf/oil_description.urdf (robot description, URDF)
Before this commit: robot oil_description, 10 links, 9 joints
Links:
- added link back_wall; collision box size=0.01 0.85 1.20; visual box size=0.01 0.85 1.20
- added link front_wall; collision box size=0.01 0.85 1.20; visual box size=0.01 0.85 1.20
- added link left_wall; collision box size=0.6 0.01 1.20; visual box size=0.6 0.01 1.20
- added link right_wall; collision box size=0.6 0.01 1.20; visual box size=0.6 0.01 1.20
Joints:
- added joint back_joint: type fixed, parent base_link, child back_wall, origin xyz=-0.32 -0.22 0.60 rpy=0 0 0, axis 0 0 0
- added joint front_joint: type fixed, parent base_link, child front_wall, origin xyz=0.32 -0.22 0.60 rpy=0 0 0, axis 0 0 0
- added joint left_joint: type fixed, parent base_link, child left_wall, origin xyz=0.0 0.22 0.60 rpy=0 0 0, axis 0 0 0
- added joint right_joint: type fixed, parent base_link, child right_wall, origin xyz=0.0 -0.65 0.60 rpy=0 0 0, axis 0 0 0
- joint joint1: limit lower=-0.34 upper=0.34 effort=0 velocity=0 -> lower=-0.42 upper=0.42 effort=0 velocity=0
- joint joint3: limit lower=-0.34 upper=0.34 effort=0 velocity=0 -> lower=-0.42 upper=0.42 effort=0 velocity=0
